File: 9-12V Power.kicad_sch (KiCad schematic)
At the start: 18 parts, among them U5 TPS54540BDDA, U6 MCP41HV51-104E/MQ

Commit message: updates to routing and digital pot
Parts:
- removed U6: MCP41HV51-104E/MQ, LEOS:QFN20_5x5MC_MCH, symbol 2026-09-23_13-25-41:MCP41HV51-104E_MQ
- added U6: MCP41100T-I/SN, LEOS:SOIC8-N_MC_MCH, symbol 2026-10-07_18-01-27:MCP41100T-I_SN
- R-4: value 25.5k -> 26.1k; Digikey RMCF0805FT25K5CT-ND -> RMCF0805FT26K1CT-ND; MPN RMCF0805FT25K5 -> RMCF0805FT26K1
Connections:
- net POT is gone; now on net GND: R-3.2
- net CS1: now also U6.1 (*CS)
- net GND: now also U6.4 (VSS), U6.5 (PA0), U6.6 (PW0), U6.7 (PB0)
- net MOSI1: now also U6.3 (SI)
- net SCK1: now also U6.2 (SCK)
- net VDD: now also U6.8 (VDD)
- no-connect marks 2 -> 1
Other:
- moved on the sheet: C-9
