File: 5V Power.kicad_sch (KiCad schematic)
At the start: 18 parts, among them U3 TPS54540BDDA

Commit message: updates to BOM and beginning of routing
Parts:
- D_1: Digikey (none) -> VS-50WQ04FNHM3GI-ND; MPN (none) -> VS-50WQ04FNHM3; Manufacturer (none) -> Vishay General Semiconductor - Diodes Division
- L_1: footprint Inductor_SMD:L_0805_2012Metric -> LEOS:IND_SRP7028A-4R7M_BRN; Digikey (none) -> SRP7028A-4R7MCT-ND; MPN (none) -> SRP7028A-4R7M; Manufacturer (none) -> Bourns Inc.
Changed lines of the file:
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@@
 			)
 		)
-		(property "Footprint" "Inductor_SMD:L_0805_2012Metric"
+		(property "Footprint" "LEOS:IND_SRP7028A-4R7M_BRN"
 			(at 171.45 72.39 0)
 			(hide yes)
@@
 		(property "Description" "Inductor"
 			(at 171.45 72.39 0)
+			(hide yes)
+			(show_name no)
+			(do_not_autoplace no)
+			(effects
+				(font
+					(size 1.27 1.27)
+				)
+			)
+		)
+		(property "Digikey" "SRP7028A-4R7MCT-ND"
+			(at 171.45 72.39 90)
+			(hide yes)
+			(show_name no)
+			(do_not_autoplace no)
+			(effects
+				(font
+					(size 1.27 1.27)
+				)
+			)
+		)
+		(property "MPN" "SRP7028A-4R7M"
+			(at 171.45 72.39 90)
+			(hide yes)
+			(show_name no)
+			(do_not_autoplace no)
+			(effects
+				(font
+					(size 1.27 1.27)
+				)
+			)
+		)
+		(property "Manufacturer" "Bourns Inc."
+			(at 171.45 72.39 90)
 			(hide yes)
 			(show_name no)
@@
 			(hide yes)
 			(show_name no)
+			(do_not_autoplace no)
+			(effects
+				(font
+					(size 1.27 1.27)
+				)
+			)
+		)
+		(property "Digikey" "VS-50WQ04FNHM3GI-ND"
+			(at 162.56 82.55 90)
+			(hide yes)
+			(show_name no)
+			(do_not_autoplace no)
+			(effects
+				(font
+					(size 1.27 1.27)
+				)
+			)
+		)
+		(property "MPN" "VS-50WQ04FNHM3"
+			(at 162.56 82.55 90)
+			(hide yes)
+			(show_name no)
+			(do_not_autoplace no)
+			(effects
+				(font
+					(size 1.27 1.27)
+				)
+			)
+		)
+		(property "Manufacturer" "Vishay General Semiconductor - Diodes Division"
+			(at 162.56 82.55 90)
+			(hide yes)
+			(show_name no)

Commit message: updates to BOM
Parts:
- removed C_9: 47u, Capacitor_SMD:C_1206_3216Metric, symbol Device:C
- removed R_1: 365k, Resistor_SMD:R_0805_2012Metric, symbol Device:R
- removed R_2: 88.7, Resistor_SMD:R_0805_2012Metric, symbol Device:R
- added TPFB5: TestPoint, TestPoint:TestPoint_Loop_D2.60mm_Drill0.9mm_Beaded, symbol Connector:TestPoint
- C_8: footprint Capacitor_SMD:C_1206_3216Metric -> LEOS:CAPAE660X600N; Digikey 4713-GMC31X5R476M25NTCT-ND -> 399-A768EB476M1VLAE042CT-ND; MPN GMC31X5R476M25NT -> A768EB476M1VLAE042; Manufacturer Cal-Chip Electronics, Inc. -> KEMET
- D_1: value 510mV -> 60V 20A; footprint Diode_SMD:D_0805_2012Metric -> Diode_THT:D_DO-201AD_P15.24mm_Horizontal; Digikey VS-50WQ04FNHM3GI-ND -> 1655-SB2060CT-ND; MPN VS-50WQ04FNHM3 -> SB2060; Manufacturer Vishay General Semiconductor - Diodes Division -> SMC Diode Solutions
Connections:
- net FB: now also TPFB5.1
- no-connect marks 0 -> 1
Other:
- note added: "Switching frequency: 643kHz"

Commit message: hid test points from bom
Parts:
- TPFB5: now left out of the parts list
Changed lines of the file:
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@@
 		(body_style 1)
 		(exclude_from_sim no)
-		(in_bom yes)
+		(in_bom no)
 		(on_board yes)
 		(in_pos_files yes)

Commit message: routing done
Parts:
- renumbered R_3 to R_1, R_4 to R_2, R_5 to R_3, R_6 to R_4
Changed lines of the file:
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@@
 		(dnp no)
 		(fields_autoplaced yes)
-		(property "Reference" "R_5"
+		(property "Reference" "R_3"
 			(at 201.93 81.2799 0)
 			(show_name no)
@@
 			(project "LEOS-F26-power"
 				(path "/3703ddf2-8141-438d-86a8-1eaec9672d0d/528ff9b0-a904-4a78-86c6-11cbf84face6"
-					(reference "R_5")
+					(reference "R_3")
 					(unit 1)
 				)
@@
 		(dnp no)
 		(fields_autoplaced yes)
-		(property "Reference" "R_3"
+		(property "Reference" "R_1"
 			(at 95.25 100.3299 0)
 			(show_name no)
@@
 			(project "LEOS-F26-power"
 				(path "/3703ddf2-8141-438d-86a8-1eaec9672d0d/528ff9b0-a904-4a78-86c6-11cbf84face6"
-					(reference "R_3")
+					(reference "R_1")
 					(unit 1)
 				)
@@
 		(dnp no)
 		(fields_autoplaced yes)
-		(property "Reference" "R_4"
+		(property "Reference" "R_2"
 			(at 157.48 101.5999 0)
 			(show_name no)
@@
 			(project "LEOS-F26-power"
 				(path "/3703ddf2-8141-438d-86a8-1eaec9672d0d/528ff9b0-a904-4a78-86c6-11cbf84face6"
-					(reference "R_4")
+					(reference "R_2")
 					(unit 1)
 				)
@@
 		(dnp no)
 		(fields_autoplaced yes)
-		(property "Reference" "R_6"
+		(property "Reference" "R_4"
 			(at 201.93 111.7599 0)
 			(show_name no)
@@
 			(project "LEOS-F26-power"
 				(path "/3703ddf2-8141-438d-86a8-1eaec9672d0d/528ff9b0-a904-4a78-86c6-11cbf84face6"
-					(reference "R_6")
+					(reference "R_4")
 					(unit 1)
 				)

Commit message: updates to BOM
Parts:
- C_1, C_2, C_3, C_4: Digikey 1276-2970-1-ND -> 1276-1248-1-ND; MPN CL21B475KOFNFNE -> CL21A475KBQNNNE
Changed lines of the file:
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@@
 			)
 		)
-		(property "Digikey" "1276-2970-1-ND"
+		(property "Digikey" "1276-1248-1-ND"
 			(at 62.23 95.25 0)
 			(hide yes)
@@
 			)
 		)
-		(property "MPN" "CL21B475KOFNFNE"
+		(property "MPN" "CL21A475KBQNNNE"
 			(at 62.23 95.25 0)
 			(hide yes)
@@
 			)
 		)
-		(property "Digikey" "1276-2970-1-ND"
+		(property "Digikey" "1276-1248-1-ND"
 			(at 46.99 95.25 0)
 			(hide yes)
@@
 			)
 		)
-		(property "MPN" "CL21B475KOFNFNE"
+		(property "MPN" "CL21A475KBQNNNE"
 			(at 46.99 95.25 0)
 			(hide yes)
@@
 			)
 		)
-		(property "Digikey" "1276-2970-1-ND"
+		(property "Digikey" "1276-1248-1-ND"
 			(at 54.61 95.25 0)
 			(hide yes)
@@
 			)
 		)
-		(property "MPN" "CL21B475KOFNFNE"
+		(property "MPN" "CL21A475KBQNNNE"
 			(at 54.61 95.25 0)
 			(hide yes)
@@
 			)
 		)
-		(property "Digikey" "1276-2970-1-ND"
+		(property "Digikey" "1276-1248-1-ND"
 			(at 69.85 95.25 0)
 			(hide yes)
@@
 			)
 		)
-		(property "MPN" "CL21B475KOFNFNE"
+		(property "MPN" "CL21A475KBQNNNE"
 			(at 69.85 95.25 0)
 			(hide yes)
