File: connectors.kicad_sch (KiCad schematic)
At the start: 7 parts, among them J1 MicroFit_1x4, J2 MicroFit_1x4

Commit message: updates to BOM and fixes for ERC
Parts:
- C6, C7: Digikey 1276-3148-1-ND -> 1276-2728-1-ND; LCSC C6142744 -> (none); MPN CL31B226MPHNNNE -> CL31A226MOCLNNC
Changed lines of the file:
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@@
 			)
 		)
-		(property "Digikey" "1276-3148-1-ND"
+		(property "Digikey" "1276-2728-1-ND"
 			(at 114.3 52.07 0)
 			(hide yes)
@@
 			)
 		)
-		(property "LCSC" "C6142744"
+		(property "LCSC" ""
 			(at 114.3 52.07 0)
 			(hide yes)
@@
 			)
 		)
-		(property "MPN" "CL31B226MPHNNNE"
+		(property "MPN" "CL31A226MOCLNNC"
 			(at 114.3 52.07 0)
 			(hide yes)
@@
 			)
 		)
-		(property "Digikey" "1276-3148-1-ND"
+		(property "Digikey" "1276-2728-1-ND"
 			(at 121.92 52.07 0)
 			(hide yes)
@@
 			)
 		)
-		(property "LCSC" "C6142744"
+		(property "LCSC" ""
 			(at 121.92 52.07 0)
 			(hide yes)
@@
 			)
 		)
-		(property "MPN" "CL31B226MPHNNNE"
+		(property "MPN" "CL31A226MOCLNNC"
 			(at 121.92 52.07 0)
 			(hide yes)

Commit message: updates to BOM
Parts:
- TP5V: renamed from TP3; Digikey 36-5000-ND -> 36-5000-ND; now in the parts list
- TPGND1: renamed from TP4; Digikey 36-5001-ND -> 36-5001-ND; now in the parts list
Changed lines of the file:
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@@
 		(body_style 1)
 		(exclude_from_sim no)
-		(in_bom no)
+		(in_bom yes)
 		(on_board yes)
-		(in_pos_files no)
+		(in_pos_files yes)
 		(dnp no)
-		(property "Reference" "TP4"
+		(property "Reference" "TPGND1"
 			(at 105.41 57.658 0)
 			(show_name no)
@@
 			)
 		)
-		(property "Digikey" "  36-5001-ND"
+		(property "Digikey" "36-5001-ND"
 			(at 104.14 55.88 0)
 			(hide yes)
@@
 			(project "LEOS-F26-power"
 				(path "/3703ddf2-8141-438d-86a8-1eaec9672d0d/341d819d-3d1a-4f8b-94f1-4c6aaa16d806"
-					(reference "TP4")
+					(reference "TPGND1")
 					(unit 1)
 				)
@@
 		(body_style 1)
 		(exclude_from_sim no)
-		(in_bom no)
+		(in_bom yes)
 		(on_board yes)
-		(in_pos_files no)
+		(in_pos_files yes)
 		(dnp no)
-		(property "Reference" "TP3"
+		(property "Reference" "TP5V"
 			(at 105.41 46.482 0)
 			(show_name no)
@@
 			)
 		)
-		(property "Digikey" "  36-5000-ND"
+		(property "Digikey" "36-5000-ND"
 			(at 104.14 48.26 0)
 			(hide yes)
@@
 			(project "LEOS-F26-power"
 				(path "/3703ddf2-8141-438d-86a8-1eaec9672d0d/341d819d-3d1a-4f8b-94f1-4c6aaa16d806"
-					(reference "TP3")
+					(reference "TP5V")
 					(unit 1)
 				)

Commit message: switching frequency
Parts:
- renumbered TP5V to TP5V1
Changed lines of the file:
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@@
 		(in_pos_files yes)
 		(dnp no)
-		(property "Reference" "TP5V"
+		(property "Reference" "TP5V1"
 			(at 105.41 46.482 0)
 			(show_name no)
@@
 			(project "LEOS-F26-power"
 				(path "/3703ddf2-8141-438d-86a8-1eaec9672d0d/341d819d-3d1a-4f8b-94f1-4c6aaa16d806"
-					(reference "TP5V")
+					(reference "TP5V1")
 					(unit 1)
 				)

Commit message: hid test points from bom
Parts:
- TP5V1, TPGND1: now left out of the parts list
Changed lines of the file:
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@@
 		(body_style 1)
 		(exclude_from_sim no)
-		(in_bom yes)
+		(in_bom no)
 		(on_board yes)
 		(in_pos_files yes)
@@
 		(body_style 1)
 		(exclude_from_sim no)
-		(in_bom yes)
+		(in_bom no)
 		(on_board yes)
 		(in_pos_files yes)

Commit message: Rename references, update symbols and schematic layout
Parts:
- R1: symbol Device:R -> Device:R_US; now in the parts list
- renumbered TP5V1 to TP3, TPGND1 to TP4
Changed lines of the file:
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@@
 	)
 	(symbol
-		(lib_id "Device:R")
+		(lib_id "Device:R_US")
 		(at 105.41 91.44 90)
 		(unit 1)
 		(body_style 1)
 		(exclude_from_sim no)
-		(in_bom no)
+		(in_bom yes)
 		(on_board yes)
-		(in_pos_files no)
+		(in_pos_files yes)
 		(dnp yes)
 		(property "Reference" "R1"
@@
 		)
 		(property "Footprint" "Resistor_THT:R_Axial_DIN0207_L6.3mm_D2.5mm_P7.62mm_Horizontal"
-			(at 105.41 93.218 90)
+			(at 105.664 90.424 90)
 			(hide yes)
 			(show_name no)
@@
 			)
 		)
-		(property "Description" "Resistor"
+		(property "Description" "Resistor, US symbol"
 			(at 105.41 91.44 0)
 			(hide yes)
@@
 		(in_bom no)
 		(on_board yes)
-		(in_pos_files yes)
+		(in_pos_files no)
 		(dnp no)
-		(property "Reference" "TPGND1"
+		(property "Reference" "TP4"
 			(at 105.41 57.658 0)
 			(show_name no)
@@
 			(project "LEOS-F26-power"
 				(path "/3703ddf2-8141-438d-86a8-1eaec9672d0d/341d819d-3d1a-4f8b-94f1-4c6aaa16d806"
-					(reference "TPGND1")
+					(reference "TP4")
 					(unit 1)
 				)
@@
 		(in_bom no)
 		(on_board yes)
-		(in_pos_files yes)
+		(in_pos_files no)
 		(dnp no)
-		(property "Reference" "TP5V1"
+		(property "Reference" "TP3"
 			(at 105.41 46.482 0)
 			(show_name no)
@@
 			(project "LEOS-F26-power"
 				(path "/3703ddf2-8141-438d-86a8-1eaec9672d0d/341d819d-3d1a-4f8b-94f1-4c6aaa16d806"
-					(reference "TP5V1")
+					(reference "TP3")
 					(unit 1)
 				)
