File: LEOS-F26-power.kicad_pcb (KiCad board)
At the start: 4 copper layers, 100 x 100 mm, 71 parts, among them J1 MicroFit_1x4, J2 MicroFit_1x4, J3 Power Input, J4 5V, J5 5V, J6 5V, J7 1-18V, J8 1-18V, J9 1-18V, U1 MCP2518FD, U2 MCP2562FD, U3 TPS54540BDDA, U4 TPS16630PWPR, U5 TPS54540BDDA, U6 MCP41100T-I/SN, Y1 40 MHz

Commit message: Rename references, update symbols and schematic layout
Parts:
- removed C-3, C-4, C_3, C_4: 4.7uF, Capacitor_SMD:C_0805_2012Metric
- removed R-3: 1.1k, Resistor_SMD:R_0805_2012Metric
- removed R-4: 26.1k, Resistor_SMD:R_0805_2012Metric
- removed TP1-18, TPFB1-18, TPFB5: TestPoint, TestPoint:TestPoint_Loop_D2.60mm_Drill0.9mm_Beaded
- removed TPGND2: GND TestPoint, TestPoint:TestPoint_Loop_D2.60mm_Drill0.9mm_Beaded
- added Rfb3: 26.1k, Resistor_SMD:R_0805_2012Metric, F.Cu at (123.0, 102.1)
- added Rfb4: 1.1k, Resistor_SMD:R_0805_2012Metric, F.Cu at (125.0, 102.1)
- Cin1: value 0.1u -> 10uF
- Cin2: value 10uF -> 0.1u
- J3: value Power Input -> XT60IPW-M
- U6: footprint LEOS:SOIC8-N_MC_MCH -> Package_SO:SOIC-8_3.9x4.9mm_P1.27mm
- moved C8 3.06 mm to (141.0, 107.0), turned to 0 degrees
- moved C9 3.00 mm to (140.9, 105.0), turned to 0 degrees
- moved L1 1.34 mm to (171.7, 127.1)
- moved Ruvlo2 1.00 mm to (161.8, 90.0)
- moved Cout3 0.90 mm to (180.0, 124.5)
- turned Cboot1 to 0 degrees
- renumbered C_1 to C10, C_2 to C11, C-9 to C12, C-1 to C8, C-2 to C9, C_5 to Cboot1, C-5 to Cboot2, C_6 to Ccomp1, C_7 to Ccomp2, C-6 to Ccomp3, C-7 to Ccomp4, C_8 to Cout3, C-8 to Cout4, CdVdt1 to Cslew1, D_1 to D1, D-1 to D2, L_1 to L1, L-1 to L2, R_1 to Rclk1, R-1 to Rclk2, R_2 to Rcomp1, R-2 to Rcomp2, R_3 to Rfb1, R_4 to Rfb2, R_ILIM1 to Rlim1, R.1 to Ruvlo1, R.2 to Ruvlo2, TP5V1 to TP3, TPGND1 to TP4
Connections:
- net +BATT renamed /E-Fuse/V_{BAT}
- net /CS1 renamed /CS
- net /MOSI1 renamed /MOSI
- net /SCK1 renamed /SCK
- net VPP renamed /VPP
- Cboot1 pad 1: Net-(D_1-K) -> Net-(U3-BOOT)
- Cboot1 pad 2: Net-(U3-BOOT) -> Net-(D1-K)
- D1 pad 1: Net-(D_1-K) -> Net-(D1-K)
- L1 pad 1: Net-(D_1-K) -> Net-(D1-K)
- U3 pad 8: Net-(D_1-K) -> Net-(D1-K)
- U5 pad 5: /1-18V Power/FB1 -> /1-18V Power/FB
- U6 pad 7: GND -> /1-18V Power/R_{adj}
Routing:
- net GND: track 75.4 -> 42.2 mm, vias 63 -> 60
- net /1-18V Power/R_{adj}: track 0.00 -> 21.9 mm
- net Net-(D_1-K): track 20.2 -> 0.00 mm, vias 2 -> 0
- net /VPP: track 35.3 -> 21.7 mm, vias 10 -> 11
- net Net-(D2-K): track 27.0 -> 13.8 mm, vias 3 -> 2
- net /1-18V Power/FB1: track 12.9 -> 0.00 mm, vias 2 -> 0
- net /5V Power/FB: track 13.7 -> 4.21 mm, vias 2 -> 0
- net /1-18V Power/FB: track 0.00 -> 4.04 mm
- net +5V: track 144.7 -> 143.8 mm
- net VDC: track 1.71 -> 1.17 mm
- net Net-(U4-DVDT): track 2.19 -> 1.69 mm
- added copper zone on F.Cu, net Net-(D1-K)
- added copper zone on F.Cu, net Net-(D2-K)
Other:
- board text added: "Battery Input"
- board text added: "Input Max 30V"
- board text removed: "Input 12-24VDC"

Commit message: ewqrngfhmhgWDFEGRHTY
Parts:
- added G***: LOGO, LOGO, F.Cu at (141.5, 131.5)

Commit message: PLEASE SPEED I NEED THIS
Parts:
- moved G*** 6.08 mm to (142.5, 125.5)
Other:
- board text added: "MY BOARD KINDA POWERLESS"

Commit message: dwedqwdqw
Other:
- board text added: "MY BOARD'S KINDA POWERLESS"
- board text removed: "MY BOARD KINDA POWERLESS"
Changed lines of the file:
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@@
 		)
 	)
-	(gr_text "MY BOARD KINDA POWERLESS"
-		(at 131.5 137.5 0)
+	(gr_text "MY BOARD'S KINDA POWERLESS"
+		(at 130.5 137.5 0)
 		(layer "F.SilkS")
 		(effects
@@
 	)
 	(zone
+		(net "/CANbus/TXCAN")
+		(layer "F.Cu")
+		(hatch none 0.1)
+		(priority 30001)
+		(attr
+			(teardrop
+				(type padvia)
+			)
+		)
+		(connect_pads yes
+			(clearance 0)
+		)
+		(min_thickness 0.0254)
+		(fill yes
+			(island_removal_mode 1)
+		)
+		(polygon
+			(pts
+				(xy 127.257842 74.128578) (xy 127.116421 73.987157) (xy 126.846465 73.974269) (xy 126.675706 74.569293)
+				(xy 126.931066 74.526066)
+			)
+		)
+	)
+	(zone
 		(net "GND")
 		(layer "F.Cu")
@@
 	)
 	(zone
+		(net "/CANbus/TXCAN")
+		(layer "F.Cu")
+		(hatch none 0.1)
+		(priority 30004)
+		(attr
+			(teardrop
+				(type padvia)
+			)
+		)
+		(connect_pads yes
+			(clearance 0)
+		)
+		(min_thickness 0.0254)
+		(fill yes
+			(island_removal_mode 1)
+		)
+		(polygon
+			(pts
+				(xy 131.116421 67.202842) (xy 131.257842 67.061421) (xy 131.045711 66.849289) (xy 130.963582 66.712597)
+				(xy 130.675707 66.620707) (xy 130.762868 67.132132) (xy 130.904289 66.990711)
+			)
+		)
+	)
+	(zone
 		(net "/VPP")
 		(layer "F.Cu")
@@
 	)
 	(zone
+		(net "/CANbus/OSC2")
+		(layer "F.Cu")
+		(hatch none 0.1)
+		(priority 30003)
+		(attr
+			(teardrop
+				(type padvia)
+			)
+		)
+		(connect_pads yes
+			(clearance 0)
+		)
+		(min_thickness 0.0254)
+		(fill yes
+			(island_removal_mode 1)
+		)
+		(polygon
+			(pts
+				(xy 131.116421 72.282843) (xy 131.257842 72.141422) (xy 130.931066 71.743934) (xy 130.675706 71.700707)
+				(xy 130.846465 72.29573)
+			)
+		)
+	)
+	(zone
 		(net "GND")
 		(layer "F.Cu")
@@
 	)
 	(zone
-		(net "/CANbus/TXCAN")
-		(layer "F.Cu")
-		(hatch none 0.1)
-		(priority 30001)
-		(attr
-			(teardrop
-				(type padvia)
-			)
-		)
-		(connect_pads yes
-			(clearance 0)
-		)
-		(min_thickness 0.0254)
-		(fill yes
-			(island_removal_mode 1)
-		)
-		(polygon
-			(pts
-				(xy 127.257842 74.128578) (xy 127.116421 73.987157) (xy 126.846465 73.974269) (xy 126.675706 74.569293)
-				(xy 126.931066 74.526066)
-			)
-		)
-	)
-	(zone
-		(net "/CANbus/OSC1")
-		(layer "F.Cu")
-		(hatch none 0.1)
-		(priority 30002)
-		(attr
-			(teardrop
-				(type padvia)
-			)
-		)
-		(connect_pads yes
-			(clearance 0)
-		)
-		(min_thickness 0.0254)
-		(fill yes
-			(island_removal_mode 1)
-		)
-		(polygon
-			(pts
-				(xy 131.116421 73.552843) (xy 131.257842 73.411422) (xy 130.931066 73.013934) (xy 130.675706 72.970707)
-				(xy 130.846465 73.56573)
-			)
-		)
-	)
-	(zone
-		(net "/CANbus/TXCAN")
+		(net "+5V")
 		(layer "F.Cu")
 		(hatch none 0.1)
-		(priority 30004)
+		(priority 30000)
 		(attr
 			(teardrop
@@
 		(polygon
 			(pts
-				(xy 131.116421 67.202842) (xy 131.257842 67.061421) (xy 131.045711 66.849289) (xy 130.963582 66.712597)
-				(xy 130.675707 66.620707) (xy 130.762868 67.132132) (xy 130.904289 66.990711)
+				(xy 124.725 71.48) (xy 124.725 71.98) (xy 125.175 72.03) (xy 126.001 71.73) (xy 125.175 71.43)
 			)
 		)
@@
 	)
 	(zone
-		(net "+5V")
-		(layer "F.Cu")
-		(hatch none 0.1)
-		(priority 30000)
-		(attr
-			(teardrop
-				(type padvia)
-			)
-		)
-		(connect_pads yes
-			(clearance 0)
-		)
-		(min_thickness 0.0254)
-		(fill yes
-			(island_removal_mode 1)
-		)
-		(polygon
-			(pts
-				(xy 124.725 71.48) (xy 124.725 71.98) (xy 125.175 72.03) (xy 126.001 71.73) (xy 125.175 71.43)
-			)
-		)
-	)
-	(zone
-		(net "/CANbus/OSC2")
-		(layer "F.Cu")
-		(hatch none 0.1)
-		(priority 30003)
-		(attr
-			(teardrop
-				(type padvia)
-			)
-		)
-		(connect_pads yes
-			(clearance 0)
-		)
-		(min_thickness 0.0254)
-		(fill yes
-			(island_removal_mode 1)
-		)
-		(polygon
-			(pts
-				(xy 131.116421 72.282843) (xy 131.257842 72.141422) (xy 130.931066 71.743934) (xy 130.675706 71.700707)
-				(xy 130.846465 72.29573)
-			)
-		)
-	)
-	(zone
 		(net "VDC")
 		(layer "F.Cu")
@@
 			)
 		)
+	)
+	(zone
+		(net "/CANbus/OSC1")
+		(layer "F.Cu")
+		(hatch none 0.1)
+		(priority 30002)
+		(attr
+			(teardrop
+				(type padvia)
+			)
+		)
+		(connect_pads yes
+			(clearance 0)
+		)
+		(min_thickness 0.0254)
+		(fill yes
+			(island_removal_mode 1)
+		)
+		(polygon
+			(pts
+				(xy 131.116421 73.552843) (xy 131.257842 73.411422) (xy 130.931066 73.013934) (xy 130.675706 72.970707)
+				(xy 130.846465 73.56573)
+			)
+		)
